File: pcb/stylus-synth.kicad_pcb (KiCad board)
At the start: 2 copper layers, 100 x 100 mm, 51 parts, among them J1 STYLUS, J2 STYLUS_PADS, J3 ST-214C, J4 SPEAKER, SW1 OCTAVE, SW2 WAVE, U2 LM386

Commit message: Finish PCB routing, add ground pour, export Gerbers
Routing:
- net +3V3: track 0.00 -> 169.4 mm, vias 0 -> 3
- net +5V: track 0.00 -> 145.2 mm, vias 0 -> 3
- net Net-(R28-Pad2): track 0.00 -> 107.4 mm, vias 0 -> 1
- net /DECAY: track 0.00 -> 59.2 mm, vias 0 -> 1
- net /BTN_WAVE: track 0.00 -> 52.1 mm
- net /VACTROL_LED: track 0.00 -> 50.8 mm
- net /AUDIO_PWM: track 0.00 -> 45.4 mm, vias 0 -> 1
- net /AUDIO_FILT: track 0.00 -> 45.1 mm
- net /SPK+: track 0.00 -> 44.7 mm
- net /AMP_OUT: track 0.00 -> 42.2 mm, vias 0 -> 1
- net /BTN_OCTAVE: track 0.00 -> 37.0 mm
- net /AMP_IN: track 0.00 -> 34.3 mm, vias 0 -> 1
- net /LPG_OUT: track 0.00 -> 34.2 mm
- net Net-(C2-Pad1): track 0.00 -> 33.3 mm
- net Net-(C9-Pad1): track 0.00 -> 26.9 mm
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- added copper zone on B.Cu, net GND
- added copper zone on F.Cu, net GND
Other:
- board text added: "2-3 VACTROL 1-2 BYPASS"
- board text added: "A"
- board text added: "A#"
- board text added: "B"
- board text added: "C"
- board text added: "C#"
- board text added: "D"
- board text added: "D#"
- board text added: "DECAY"
- board text added: "E"
- board text added: "F"
- board text added: "F#"
- board text added: "G"
- board text added: "G#"
- board text added: "PHONES"
- board text added: "R1-R21 = 1k"
- board text added: "Stylus Synthesizer Hack Club Half Life Week 3"
- board text added: "VOL"
